Commit message: made finger joints mimic of shared servo joint

File: rh_p12_rn_description/urdf/rh_p12_rn.urdf.xacro (robot description, xacro)
@@ -1,13 +1,13 @@
 <?xml version="1.0"?>
 <robot name="rh_p12_rn" xmlns:xacro="http://ros.org/wiki/xacro">
-  <!-- some parameters -->
   <xacro:macro name="rh_p12_rn_macro" params="parent prefix reflect *origin">
-    <joint name="${prefix}_rh_p12_rn_joint" type="fixed">
+    <!-- Base Joint -->
+    <joint name="${prefix}_base_joint" type="fixed">
       <xacro:insert_block name="origin"/>
       <parent link="${parent}"/>
-      <child link="${prefix}_rh_p12_rn_base"/>
-    </joint>
-    <!-- base -->
-    <link name="${prefix}_rh_p12_rn_base">
+      <child link="${prefix}_base"/>
+    </joint>
+    <!-- Base -->
+    <link name="${prefix}_base">
       <collision>
         <origin xyz="0 0 0" rpy="0 0 0"/>
@@ -30,21 +30,32 @@
       </inertial>
     </link>
-    <gazebo reference="${prefix}_rh_p12_rn_base">
-      <mu1>0.2</mu1>
-      <mu2>0.2</mu2>
-      <material>Gazebo/Grey</material>
-    </gazebo>
-    <!-- Joint -->
-    <joint name="${prefix}_rh_p12_rn" type="revolute">
-      <parent link="${prefix}_rh_p12_rn_base"/>
-      <child link="${prefix}_rh_p12_rn_r1"/>
+    <gazebo reference="${prefix}_base">
+      <mu1>0.2</mu1>
+      <mu2>0.2</mu2>
+      <material>Gazebo/Grey</material>
+    </gazebo>
+    <!-- Finger Motor Joint -->
+    <joint name="${prefix}_finger_servo_joint" type="revolute">
+        <origin xyz="0 0.0 0" rpy="0 0 0" />
+        <axis xyz="1 0 0" />
+        <limit lower="0" upper="1.1" effort="4" velocity="5" />
+        <parent link="${prefix}_base" />
+        <child link="${prefix}_finger_servo_link" />
+    </joint>
+    <link name="${prefix}_finger_servo_link">
+    </link>
+    <!-- Right Joint 1-->
+    <joint name="${prefix}_joint_r1" type="revolute">
+      <parent link="${prefix}_base"/>
+      <child link="${prefix}_link_r1"/>
       <origin xyz="0.0 0.008 0.048" rpy="0 0 0"/>
       <axis xyz="1 0 0"/>
       <limit velocity="6.5" effort="1000" lower="0.0" upper="1.1" />
       <dynamics damping="0.7"/>
-    </joint>
-    <transmission name="${prefix}_tran_r1">
-      <type>transmission_interface/SimpleTransmission</type>
-      <joint name="${prefix}_rh_p12_rn">
+      <mimic joint="${prefix}_finger_servo_joint" multiplier="1" offset="0"/>
+    </joint>
+    <transmission name="${prefix}_transmission_r1">
+      <type>transmission_interface/SimpleTransmission</type>
+      <joint name="${prefix}_join_r1">
         <hardwareInterface>hardware_interface/PositionJointInterface</hardwareInterface>
       </joint>
@@ -54,6 +65,6 @@
       </actuator>
     </transmission>
-    <!-- rh_p12_rn_r1 -->
-    <link name="${prefix}_rh_p12_rn_r1">
+    <!-- Left Link 1 -->
+    <link name="${prefix}_link_r1">
       <collision>
         <origin xyz="0 0 0" rpy="0 0 0"/>
@@ -76,5 +87,5 @@
       </inertial>
     </link>
-    <gazebo reference="${prefix}_rh_p12_rn_r1">
+    <gazebo reference="${prefix}_r1">
       <mu1>0.2</mu1>
       <mu2>0.2</mu2>
@@ -82,15 +93,16 @@
     </gazebo>
     <!-- Right Joint 2 -->
-    <joint name="${prefix}_rh_r2" type="revolute">
-      <parent link="${prefix}_rh_p12_rn_r1"/>
-      <child link="${prefix}_rh_p12_rn_r2"/>
+    <joint name="${prefix}_joint_r2" type="revolute">
+      <parent link="${prefix}_link_r1"/>
+      <child link="${prefix}_link_r2"/>
       <origin xyz="0.0 0.0493634 0.0285" rpy="0 0 0"/>
       <axis xyz="-1 0 0"/>
       <limit velocity="6.5" effort="1000" lower="0.0" upper="1.0" />
       <dynamics damping="0.7"/>
-    </joint>
-    <transmission name="${prefix}_tran_r2">
-      <type>transmission_interface/SimpleTransmission</type>
-      <joint name="${prefix}_rh_r2">
+      <mimic joint="${prefix}_finger_servo_joint" multiplier="0.909" offset="0"/>s
+    </joint>
+    <transmission name="${prefix}_transmission_r2">
+      <type>transmission_interface/SimpleTransmission</type>
+      <joint name="${prefix}_joint_r2">
         <hardwareInterface>hardware_interface/PositionJointInterface</hardwareInterface>
       </joint>
@@ -100,6 +112,6 @@
       </actuator>
     </transmission>
-    <!-- rh_p12_rn_r2 -->
-    <link name="${prefix}_rh_p12_rn_r2">
+    <!-- Right Link 2 -->
+    <link name="${prefix}_link_r2">
       <collision>
         <origin xyz="0 0 0" rpy="0 0 0"/>
@@ -122,5 +134,5 @@
       </inertial>
     </link>
-    <gazebo reference="${prefix}_rh_p12_rn_r2">
+    <gazebo reference="${prefix}_r2">
       <mu1>0.2</mu1>
       <mu2>0.2</mu2>
@@ -128,15 +140,16 @@
     </gazebo>
     <!-- Left Joint 1 -->
-    <joint name="${prefix}_rh_l1" type="revolute">
-      <parent link="${prefix}_rh_p12_rn_base"/>
-      <child link="${prefix}_rh_p12_rn_l1"/>
+    <joint name="${prefix}_joint_l1" type="revolute">
+      <parent link="${prefix}_base"/>
+      <child link="${prefix}_link_l1"/>
       <origin xyz="0.0 -0.008 0.048" rpy="0 0 0"/>
       <axis xyz="-1 0 0"/>
       <limit velocity="6.5" effort="1000" lower="0.0" upper="1.1" />
       <dynamics damping="0.7"/>
-    </joint>
-    <transmission name="${prefix}_tran_l1">
-      <type>transmission_interface/SimpleTransmission</type>
-      <joint name="${prefix}_rh_l1">
+      <mimic joint="${prefix}_finger_servo_joint" multiplier="1" offset="0"/>
+    </joint>
+    <transmission name="${prefix}_transmission_l1">
+      <type>transmission_interface/SimpleTransmission</type>
+      <joint name="${prefix}_joint_l1">
         <hardwareInterface>hardware_interface/PositionJointInterface</hardwareInterface>
       </joint>
@@ -146,6 +159,6 @@
       </actuator>
     </transmission>
-    <!-- rh_p12_rn_l1 -->
-    <link name="${prefix}_rh_p12_rn_l1">
+    <!-- Left Link 1 -->
+    <link name="${prefix}_link_l1">
       <collision>
         <origin xyz="0 0 0" rpy="0 0 0"/>
@@ -168,5 +181,5 @@
       </inertial>
     </link>
-    <gazebo reference="${prefix}_rh_p12_rn_l1">
+    <gazebo reference="${prefix}_link_l1">
       <mu1>0.2</mu1>
       <mu2>0.2</mu2>
@@ -174,15 +187,16 @@
     </gazebo>
     <!-- Left Joint 2 -->
-    <joint name="${prefix}_rh_l2" type="revolute">
-      <parent link="${prefix}_rh_p12_rn_l1"/>
-      <child link="${prefix}_rh_p12_rn_l2"/>
+    <joint name="${prefix}_joint_l2" type="revolute">
+      <parent link="${prefix}_link_l1"/>
+      <child link="${prefix}_link_l2"/>
       <origin xyz="0.0 -0.0493634 0.0285" rpy="0 0 0"/>
       <axis xyz="1 0 0"/>
       <limit velocity="6.5" effort="1000" lower="0.0" upper="1.0" />
       <dynamics damping="0.7"/>
-    </joint>
-    <transmission name="${prefix}_tran_l2">
-      <type>transmission_interface/SimpleTransmission</type>
-      <joint name="${prefix}_rh_l2">
+      <mimic joint="${prefix}_finger_servo_joint" multiplier="0.909" offset="0"/>
+    </joint>
+    <transmission name="${prefix}_transmission_l2">
+      <type>transmission_interface/SimpleTransmission</type>
+      <joint name="${prefix}_joint_l2">
         <hardwareInterface>hardware_interface/PositionJointInterface</hardwareInterface>
       </joint>
@@ -192,6 +206,6 @@
       </actuator>
     </transmission>
-    <!-- rh_p12_rn_l2 -->
-    <link name="${prefix}_rh_p12_rn_l2">
+    <!-- Left Link 2 -->
+    <link name="${prefix}_link_l2">
       <collision>
         <origin xyz="0 0 0" rpy="0 0 0"/>
@@ -214,5 +228,5 @@
       </inertial>
     </link>
-    <gazebo reference="${prefix}_rh_p12_rn_l2">
+    <gazebo reference="${prefix}_link_l2">
       <mu1>0.2</mu1>
       <mu2>0.2</mu2>

Commit message: renamed servo joint added gazebo mimic plugins

File: rh_p12_rn_description/urdf/rh_p12_rn.urdf.xacro (robot description, xacro)
@@ -36,12 +36,22 @@
     </gazebo>
     <!-- Finger Motor Joint -->
-    <joint name="${prefix}_finger_servo_joint" type="revolute">
+    <joint name="${prefix}_servo_joint" type="revolute">
         <origin xyz="0 0.0 0" rpy="0 0 0" />
         <axis xyz="1 0 0" />
-        <limit lower="0" upper="1.1" effort="4" velocity="5" />
+        <limit lower="0" upper="1.15" effort="4" velocity="5" />
         <parent link="${prefix}_base" />
-        <child link="${prefix}_finger_servo_link" />
-    </joint>
-    <link name="${prefix}_finger_servo_link">
+        <child link="${prefix}_servo_link" />
+    </joint>
+    <transmission name="${prefix}_servo_joint_transmission">
+      <type>transmission_interface/SimpleTransmission</type>
+      <joint name="${prefix}_servo_joint">
+        <hardwareInterface>hardware_interface/EffortJointInterface</hardwareInterface>
+      </joint>
+      <actuator name="${prefix}_servo_joint_motor">
+        <hardwareInterface>hardware_interface/EffortJointInterface</hardwareInterface>
+        <mechanicalReduction>1</mechanicalReduction>
+      </actuator>
+    </transmission>
+    <link name="${prefix}_servo_link">
     </link>
     <!-- Right Joint 1-->
@@ -53,9 +63,19 @@
       <limit velocity="6.5" effort="1000" lower="0.0" upper="1.1" />
       <dynamics damping="0.7"/>
-      <mimic joint="${prefix}_finger_servo_joint" multiplier="1" offset="0"/>
-    </joint>
-    <transmission name="${prefix}_transmission_r1">
-      <type>transmission_interface/SimpleTransmission</type>
-      <joint name="${prefix}_join_r1">
+      <mimic joint="${prefix}_servo_joint" multiplier="1" offset="0"/>
+    </joint>
+    <gazebo>
+      <plugin name="mimic_${prefix}_joint_r1" filename="libroboticsgroup_gazebo_mimic_joint_plugin.so">
+        <joint>${prefix}_servo_joint</joint>
+        <mimicJoint>${prefix}_joint_r1</mimicJoint>
+        <multiplier>1</multiplier>
+        <offset>0</offset>
+        <maxEffort>4</maxEffort>
+        <hasPID/>
+      </plugin>
+    </gazebo>
+<!--    <transmission name="${prefix}_transmission_r1">
+      <type>transmission_interface/SimpleTransmission</type>
+      <joint name="${prefix}_joint_r1">
         <hardwareInterface>hardware_interface/PositionJointInterface</hardwareInterface>
       </joint>
@@ -64,5 +84,5 @@
         <mechanicalReduction>1</mechanicalReduction>
       </actuator>
-    </transmission>
+    </transmission>-->
     <!-- Left Link 1 -->
     <link name="${prefix}_link_r1">
@@ -100,7 +120,17 @@
       <limit velocity="6.5" effort="1000" lower="0.0" upper="1.0" />
       <dynamics damping="0.7"/>
-      <mimic joint="${prefix}_finger_servo_joint" multiplier="0.909" offset="0"/>s
-    </joint>
-    <transmission name="${prefix}_transmission_r2">
+      <mimic joint="${prefix}_servo_joint" multiplier="0.909" offset="0"/>s
+    </joint>
+    <gazebo>
+      <plugin name="mimic_${prefix}_joint_r2" filename="libroboticsgroup_gazebo_mimic_joint_plugin.so">
+        <joint>${prefix}_servo_joint</joint>
+        <mimicJoint>${prefix}_joint_r2</mimicJoint>
+        <multiplier>0.909</multiplier>
+        <offset>0</offset>
+        <maxEffort>4</maxEffort>
+        <hasPID/>
+      </plugin>
+    </gazebo>
+<!--    <transmission name="${prefix}_transmission_r2">
       <type>transmission_interface/SimpleTransmission</type>
       <joint name="${prefix}_joint_r2">
@@ -111,5 +141,5 @@
         <mechanicalReduction>1</mechanicalReduction>
       </actuator>
-    </transmission>
+    </transmission>-->
     <!-- Right Link 2 -->
     <link name="${prefix}_link_r2">
@@ -147,7 +177,17 @@
       <limit velocity="6.5" effort="1000" lower="0.0" upper="1.1" />
       <dynamics damping="0.7"/>
-      <mimic joint="${prefix}_finger_servo_joint" multiplier="1" offset="0"/>
-    </joint>
-    <transmission name="${prefix}_transmission_l1">
+      <mimic joint="${prefix}_servo_joint" multiplier="1" offset="0"/>
+    </joint>
+    <gazebo>
+      <plugin name="mimic_${prefix}_joint_l1" filename="libroboticsgroup_gazebo_mimic_joint_plugin.so">
+        <joint>${prefix}_servo_joint</joint>
+        <mimicJoint>${prefix}_joint_l1</mimicJoint>
+        <multiplier>1</multiplier>
+        <offset>0</offset>
+        <maxEffort>4</maxEffort>
+        <hasPID/>
+      </plugin>
+    </gazebo>
+<!--    <transmission name="${prefix}_transmission_l1">
       <type>transmission_interface/SimpleTransmission</type>
       <joint name="${prefix}_joint_l1">
@@ -158,5 +198,5 @@
         <mechanicalReduction>1</mechanicalReduction>
       </actuator>
-    </transmission>
+    </transmission>-->
     <!-- Left Link 1 -->
     <link name="${prefix}_link_l1">
@@ -194,7 +234,17 @@
       <limit velocity="6.5" effort="1000" lower="0.0" upper="1.0" />
       <dynamics damping="0.7"/>
-      <mimic joint="${prefix}_finger_servo_joint" multiplier="0.909" offset="0"/>
-    </joint>
-    <transmission name="${prefix}_transmission_l2">
+      <mimic joint="${prefix}_servo_joint" multiplier="0.909" offset="0"/>
+    </joint>
+    <gazebo>
+      <plugin name="mimic_${prefix}_joint_l2" filename="libroboticsgroup_gazebo_mimic_joint_plugin.so">
+        <joint>${prefix}_servo_joint</joint>
+        <mimicJoint>${prefix}_joint_l2</mimicJoint>
+        <multiplier>0.909</multiplier>
+        <offset>0</offset>
+        <maxEffort>4</maxEffort>
+        <hasPID/>
+      </plugin>
+    </gazebo>
+<!--    <transmission name="${prefix}_transmission_l2">
       <type>transmission_interface/SimpleTransmission</type>
       <joint name="${prefix}_joint_l2">
@@ -205,5 +255,5 @@
         <mechanicalReduction>1</mechanicalReduction>
       </actuator>
-    </transmission>
+    </transmission>-->
     <!-- Left Link 2 -->
     <link name="${prefix}_link_l2">

Commit message: fixed gripper in simulation by adding a small inertia to the gripper servo joint

File: rh_p12_rn_description/urdf/rh_p12_rn.urdf.xacro (robot description, xacro)
@@ -54,4 +54,9 @@
     </transmission>
     <link name="${prefix}_servo_link">
+      <inertial>
+        <origin xyz="0 0 0" rpy="0 0 0" />
+        <mass value="0.01" />
+        <inertia ixx="1.0e-6" ixy="0.0" ixz="0.0" iyy="1.0e-6" iyz="0.0" izz="1.0e-6" />
+      </inertial>
     </link>
     <!-- Right Joint 1-->

Commit message: Add convex versions of geometries and use for collision tags

File: rh_p12_rn_description/urdf/rh_p12_rn.urdf.xacro (robot description, xacro)
@@ -13,5 +13,5 @@
         <origin xyz="0 0 0" rpy="0 0 0"/>
         <geometry>
-          <mesh filename="package://rh_p12_rn_description/meshes/base.stl" scale="0.001 0.001 0.001"/>
+          <mesh filename="package://rh_p12_rn_description/meshes/base_convex.stl" scale="0.001 0.001 0.001"/>
         </geometry>
       </collision>
@@ -95,5 +95,5 @@
         <origin xyz="0 0 0" rpy="0 0 0"/>
         <geometry>
-          <mesh filename="package://rh_p12_rn_description/meshes/r1.stl" scale="0.001 0.001 0.001"/>
+          <mesh filename="package://rh_p12_rn_description/meshes/r1_convex.stl" scale="0.001 0.001 0.001"/>
         </geometry>
       </collision>
@@ -152,5 +152,5 @@
         <origin xyz="0 0 0" rpy="0 0 0"/>
         <geometry>
-          <mesh filename="package://rh_p12_rn_description/meshes/r2.stl" scale="0.001 0.001 0.001"/>
+          <mesh filename="package://rh_p12_rn_description/meshes/r2_convex.stl" scale="0.001 0.001 0.001"/>
         </geometry>
       </collision>
@@ -209,5 +209,5 @@
         <origin xyz="0 0 0" rpy="0 0 0"/>
         <geometry>
-          <mesh filename="package://rh_p12_rn_description/meshes/l1.stl" scale="0.001 0.001 0.001"/>
+          <mesh filename="package://rh_p12_rn_description/meshes/l1_convex.stl" scale="0.001 0.001 0.001"/>
         </geometry>
       </collision>
@@ -266,5 +266,5 @@
         <origin xyz="0 0 0" rpy="0 0 0"/>
         <geometry>
-          <mesh filename="package://rh_p12_rn_description/meshes/l2.stl" scale="0.001 0.001 0.001"/>
+          <mesh filename="package://rh_p12_rn_description/meshes/l2_convex.stl" scale="0.001 0.001 0.001"/>
         </geometry>
       </collision>

Commit message: Fix inertias to be plausible

File: rh_p12_rn_description/urdf/rh_p12_rn.urdf.xacro (robot description, xacro)
@@ -2,4 +2,5 @@
 <robot name="rh_p12_rn" xmlns:xacro="http://ros.org/wiki/xacro">
   <xacro:macro name="rh_p12_rn_macro" params="parent prefix reflect *origin">
+    <xacro:include filename="$(find hector_xacro_tools)/urdf/inertia_tensors.urdf.xacro" />
     <!-- Base Joint -->
     <joint name="${prefix}_base_joint" type="fixed">
@@ -23,10 +24,15 @@
         <material name="grey"/>
       </visual>
+      <!--
       <inertial>
         <origin xyz="0.000 0.000 0.032" rpy="0 0 0"/>
-        <mass value="0.236"/>
+        <mass value="0.236"/>-->
         <!--<inertia ixx="0.00017" ixy="0.0" ixz="0.0" iyy="0.00011" iyz="0.0" izz="0.00017" />-->
-        <inertia ixx="1.0" ixy="0.0" ixz="0.0" iyy="1.0" iyz="0.0" izz="1.0" />
+       <!-- <inertia ixx="1.0" ixy="0.0" ixz="0.0" iyy="1.0" iyz="0.0" izz="1.0" />
       </inertial>
+      -->
+      <xacro:inertial_cuboid_with_pose mass="0.236" x_length="0.08" y_length="0.08" z_length="0.08" >
+            <origin xyz="0.000 0.000 0.032" rpy="0 0 0" />
+      </xacro:inertial_cuboid_with_pose>
     </link>
     <gazebo reference="${prefix}_base">
@@ -54,9 +60,13 @@
     </transmission>
     <link name="${prefix}_servo_link">
-      <inertial>
+      <!--<inertial>
         <origin xyz="0 0 0" rpy="0 0 0" />
         <mass value="0.01" />
         <inertia ixx="1.0e-6" ixy="0.0" ixz="0.0" iyy="1.0e-6" iyz="0.0" izz="1.0e-6" />
       </inertial>
+      -->
+      <xacro:inertial_cuboid_with_pose mass="0.01" x_length="0.04" y_length="0.04" z_length="0.04" >
+        <origin xyz="0.0 0.0 0.0" rpy="0 0 0" />
+      </xacro:inertial_cuboid_with_pose>
     </link>
     <!-- Right Joint 1-->
@@ -66,6 +76,6 @@
       <origin xyz="0.0 0.008 0.048" rpy="0 0 0"/>
       <axis xyz="1 0 0"/>
-      <limit velocity="6.5" effort="1000" lower="0.0" upper="1.1" />
-      <dynamics damping="0.7"/>
+      <limit velocity="6.5" effort="10" lower="0.0" upper="1.1" />
+      <!--<dynamics damping="0.7"/>--> <!--WARNING: This makes Gazebo sim explode-->
       <mimic joint="${prefix}_servo_joint" multiplier="1" offset="0"/>
     </joint>
@@ -105,10 +115,15 @@
         <material name="grey"/>
       </visual>
+      <!--
       <inertial>
         <origin xyz="0.000 0.034 0.004" rpy="0 0 0"/>
-        <mass value="0.068"/>
+        <mass value="0.068"/>-->
         <!--<inertia ixx="0.00004" ixy="0.0" ixz="0.0" iyy="0.00002" iyz="-0.00001" izz="0.00002" />-->
-        <inertia ixx="1.0" ixy="0.0" ixz="0.0" iyy="1.0" iyz="0.0" izz="1.0" />
+        <!--<inertia ixx="1.0" ixy="0.0" ixz="0.0" iyy="1.0" iyz="0.0" izz="1.0" />
       </inertial>
+      -->
+      <xacro:inertial_cuboid_with_pose mass="0.068" x_length="0.04" y_length="0.04" z_length="0.04" >
+        <origin xyz="0.000 0.034 0.004" rpy="0 0 0" />
+      </xacro:inertial_cuboid_with_pose>
     </link>
     <gazebo reference="${prefix}_link_r1">
@@ -123,6 +138,6 @@
       <origin xyz="0.0 0.0493634 0.0285" rpy="0 0 0"/>
       <axis xyz="-1 0 0"/>
-      <limit velocity="6.5" effort="1000" lower="0.0" upper="1.0" />
-      <dynamics damping="0.7"/>
+      <limit velocity="6.5" effort="10" lower="0.0" upper="1.0" />
+      <!--<dynamics damping="0.7"/>--> <!--WARNING: This makes Gazebo sim explode-->
       <mimic joint="${prefix}_servo_joint" multiplier="0.909" offset="0"/>s
     </joint>
@@ -162,10 +177,14 @@
         <material name="grey"/>
       </visual>
+      <!--
       <inertial>
         <origin xyz="0.000 0.006 0.011" rpy="0 0 0"/>
-        <mass value="0.022"/>
+        <mass value="0.022"/>-->
         <!--<inertia ixx="0.0" ixy="0.0" ixz="0.0" iyy="0.00001" iyz="0.0" izz="0.0" />-->
-        <inertia ixx="1.0" ixy="0.0" ixz="0.0" iyy="1.0" iyz="0.0" izz="1.0" />
-      </inertial>
+      <!--<inertia ixx="1.0" ixy="0.0" ixz="0.0" iyy="1.0" iyz="0.0" izz="1.0" />
+      </inertial>-->
+      <xacro:inertial_cuboid_with_pose mass="0.022" x_length="0.04" y_length="0.04" z_length="0.04" >
+        <origin xyz="0.000 0.006 0.011" rpy="0 0 0" />
+      </xacro:inertial_cuboid_with_pose>
     </link>
     <gazebo reference="${prefix}_link_r2">
@@ -180,6 +199,6 @@
       <origin xyz="0.0 -0.008 0.048" rpy="0 0 0"/>
       <axis xyz="-1 0 0"/>
-      <limit velocity="6.5" effort="1000" lower="0.0" upper="1.1" />
-      <dynamics damping="0.7"/>
+      <limit velocity="6.5" effort="10" lower="0.0" upper="1.1" />
+      <!--<dynamics damping="0.7"/>--> <!--WARNING: This makes Gazebo sim explode-->
       <mimic joint="${prefix}_servo_joint" multiplier="1" offset="0"/>
     </joint>
@@ -219,10 +238,14 @@
         <material name="grey"/>
       </visual>
+      <!--
       <inertial>
         <origin xyz="0.000 -0.034 0.004" rpy="0 0 0"/>
-        <mass value="0.068"/>
+        <mass value="0.068"/>-->
         <!--<inertia ixx="0.00004" ixy="0.0" ixz="0.0" iyy="0.00002" iyz="0.00001" izz="0.00002" />-->
-        <inertia ixx="1.0" ixy="0.0" ixz="0.0" iyy="1.0" iyz="0.0" izz="1.0" />
-      </inertial>
+        <!--<inertia ixx="1.0" ixy="0.0" ixz="0.0" iyy="1.0" iyz="0.0" izz="1.0" />
+      </inertial>-->
+      <xacro:inertial_cuboid_with_pose mass="0.068" x_length="0.04" y_length="0.04" z_length="0.04" >
+        <origin xyz="0.000 -0.034 0.004" rpy="0 0 0" />
+      </xacro:inertial_cuboid_with_pose>
     </link>
     <gazebo reference="${prefix}_link_l1">
@@ -237,6 +260,6 @@
       <origin xyz="0.0 -0.0493634 0.0285" rpy="0 0 0"/>
       <axis xyz="1 0 0"/>
-      <limit velocity="6.5" effort="1000" lower="0.0" upper="1.0" />
-      <dynamics damping="0.7"/>
+      <limit velocity="6.5" effort="10" lower="0.0" upper="1.0" />
+      <!--<dynamics damping="0.7"/>--> <!--WARNING: This makes Gazebo sim explode-->s
       <mimic joint="${prefix}_servo_joint" multiplier="0.909" offset="0"/>
     </joint>
@@ -276,10 +299,14 @@
         <material name="grey"/>
       </visual>
+      <!--
       <inertial>
         <origin xyz="0.000 -0.006 0.011" rpy="0 0 0"/>
-        <mass value="0.022"/>
+        <mass value="0.022"/>-->
         <!--<inertia ixx="0.0" ixy="0.0" ixz="0.0" iyy="0.00001" iyz="0.0" izz="0.0" />-->
-        <inertia ixx="1.0" ixy="0.0" ixz="0.0" iyy="1.0" iyz="0.0" izz="1.0" />
-      </inertial>
+        <!--<inertia ixx="1.0" ixy="0.0" ixz="0.0" iyy="1.0" iyz="0.0" izz="1.0" />
+      </inertial>-->
+      <xacro:inertial_cuboid_with_pose mass="0.022" x_length="0.04" y_length="0.04" z_length="0.04" >
+        <origin xyz="0.000 -0.006 0.011" rpy="0 0 0" />
+      </xacro:inertial_cuboid_with_pose>
     </link>
     <gazebo reference="${prefix}_link_l2">
