Commit message: Add links for grasp planning (main and tip)

File: rh_p12_rn_description/urdf/rh_p12_rn.urdf.xacro (robot description, xacro)
@@ -310,4 +310,18 @@
       </xacro:inertial_cuboid_with_pose>
     </link>
+    <joint name="gripper_grasp_main_joint" type="fixed">
+      <origin xyz="0.0 0 0.11" rpy="${M_PI} ${-M_PI*0.5} ${M_PI*0}" />
+      <parent link="${prefix}_base" />
+      <child link="gripper_grasp_main_link" />
+    </joint>
+    <link name="gripper_grasp_main_link">
+    </link>
+    <joint name="gripper_grasp_tip_joint" type="fixed">
+      <origin xyz="0.0 0 0.15" rpy="${M_PI} ${-M_PI*0.5} ${M_PI*0}" />
+      <parent link="${prefix}_base" />
+      <child link="gripper_grasp_tip_link" />
+    </joint>
+    <link name="gripper_grasp_tip_link">
+    </link>
     <gazebo reference="${prefix}_link_l2">
       <mu1>0.2</mu1>

Commit message: removed inverted axes

File: rh_p12_rn_description/urdf/rh_p12_rn.urdf.xacro (robot description, xacro)
@@ -136,6 +136,6 @@
       <parent link="${prefix}_link_r1"/>
       <child link="${prefix}_link_r2"/>
-      <origin xyz="0.0 0.0493634 0.0285" rpy="0 0 0"/>
-      <axis xyz="-1 0 0"/>
+      <origin xyz="0.0 0.0493634 0.0285" rpy="0 0 ${M_PI}"/>
+      <axis xyz="1 0 0"/>
       <limit velocity="6.5" effort="10" lower="0.0" upper="1.0" />
       <!--<dynamics damping="0.7"/>--> <!--WARNING: This makes Gazebo sim explode-->
@@ -165,5 +165,5 @@
     <link name="${prefix}_link_r2">
       <collision>
-        <origin xyz="0 0 0" rpy="0 0 0"/>
+        <origin xyz="0 0 0" rpy="0 0 ${M_PI}"/>
         <geometry>
           <mesh filename="package://rh_p12_rn_description/meshes/r2_convex.stl" scale="0.001 0.001 0.001"/>
@@ -171,5 +171,5 @@
       </collision>
       <visual>
-        <origin xyz="0 0 0" rpy="0 0 0"/>
+        <origin xyz="0 0 0" rpy="0 0 ${M_PI}"/>
         <geometry>
           <mesh filename="package://rh_p12_rn_description/meshes/r2.stl" scale="0.001 0.001 0.001"/>
@@ -185,5 +185,5 @@
       </inertial>-->
       <xacro:inertial_cuboid_with_pose mass="0.022" x_length="0.04" y_length="0.04" z_length="0.04" >
-        <origin xyz="0.000 0.006 0.011" rpy="0 0 0" />
+        <origin xyz="0.000 -0.006 0.011" rpy="0 0 0" />
       </xacro:inertial_cuboid_with_pose>
     </link>
@@ -197,6 +197,6 @@
       <parent link="${prefix}_base"/>
       <child link="${prefix}_link_l1"/>
-      <origin xyz="0.0 -0.008 0.048" rpy="0 0 0"/>
-      <axis xyz="-1 0 0"/>
+      <origin xyz="0.0 -0.008 0.048" rpy="0 0 ${M_PI}"/>
+      <axis xyz="1 0 0"/>
       <limit velocity="6.5" effort="10" lower="0.0" upper="1.1" />
       <!--<dynamics damping="0.7"/>--> <!--WARNING: This makes Gazebo sim explode-->
@@ -226,5 +226,5 @@
     <link name="${prefix}_link_l1">
       <collision>
-        <origin xyz="0 0 0" rpy="0 0 0"/>
+        <origin xyz="0 0 0" rpy="0 0 ${M_PI}"/>
         <geometry>
           <mesh filename="package://rh_p12_rn_description/meshes/l1_convex.stl" scale="0.001 0.001 0.001"/>
@@ -232,5 +232,5 @@
       </collision>
       <visual>
-        <origin xyz="0 0 0" rpy="0 0 0"/>
+        <origin xyz="0 0 0" rpy="0 0 ${M_PI}"/>
         <geometry>
           <mesh filename="package://rh_p12_rn_description/meshes/l1.stl" scale="0.001 0.001 0.001"/>
@@ -246,5 +246,5 @@
       </inertial>-->
       <xacro:inertial_cuboid_with_pose mass="0.068" x_length="0.04" y_length="0.04" z_length="0.04" >
-        <origin xyz="0.000 -0.034 0.004" rpy="0 0 0" />
+        <origin xyz="0.000 0.034 0.004" rpy="0 0 0" />
       </xacro:inertial_cuboid_with_pose>
     </link>
@@ -258,5 +258,5 @@
       <parent link="${prefix}_link_l1"/>
       <child link="${prefix}_link_l2"/>
-      <origin xyz="0.0 -0.0493634 0.0285" rpy="0 0 0"/>
+      <origin xyz="0.0 0.0493634 0.0285" rpy="0 0 ${M_PI}"/>
       <axis xyz="1 0 0"/>
       <limit velocity="6.5" effort="10" lower="0.0" upper="1.0" />

Commit message: changed the color to match the real gripper

File: rh_p12_rn_description/urdf/rh_p12_rn.urdf.xacro (robot description, xacro)
@@ -39,5 +39,5 @@
       <mu1>0.2</mu1>
       <mu2>0.2</mu2>
-      <material>Gazebo/Grey</material>
+      <material>Gazebo/DarkGrey</material>
     </gazebo>
     <!-- Finger Motor Joint -->
@@ -130,5 +130,5 @@
       <mu1>0.2</mu1>
       <mu2>0.2</mu2>
-      <material>Gazebo/Grey</material>
+      <material>Gazebo/DarkGrey</material>
     </gazebo>
     <!-- Right Joint 2 -->
@@ -191,5 +191,5 @@
       <mu1>0.2</mu1>
       <mu2>0.2</mu2>
-      <material>Gazebo/Grey</material>
+      <material>Gazebo/DarkGrey</material>
     </gazebo>
     <!-- Left Joint 1 -->
@@ -252,5 +252,5 @@
       <mu1>0.2</mu1>
       <mu2>0.2</mu2>
-      <material>Gazebo/Grey</material>
+      <material>Gazebo/DarkGrey</material>
     </gazebo>
     <!-- Left Joint 2 -->
@@ -327,5 +327,5 @@
       <mu1>0.2</mu1>
       <mu2>0.2</mu2>
-      <material>Gazebo/Grey</material>
+      <material>Gazebo/DarkGrey</material>
     </gazebo>
   </xacro:macro>

Commit message: cleanup

File: rh_p12_rn_description/urdf/rh_p12_rn.urdf.xacro (robot description, xacro)
@@ -90,14 +90,4 @@
       </plugin>
     </gazebo>
-<!--    <transmission name="${prefix}_transmission_r1">
-      <type>transmission_interface/SimpleTransmission</type>
-      <joint name="${prefix}_joint_r1">
-        <hardwareInterface>hardware_interface/PositionJointInterface</hardwareInterface>
-      </joint>
-      <actuator name="${prefix}_motor_r1">
-        <hardwareInterface>hardware_interface/PositionJointInterface</hardwareInterface>
-        <mechanicalReduction>1</mechanicalReduction>
-      </actuator>
-    </transmission>-->
     <!-- Right Link 1 -->
     <link name="${prefix}_link_r1">
@@ -152,14 +142,4 @@
       </plugin>
     </gazebo>
-<!--    <transmission name="${prefix}_transmission_r2">
-      <type>transmission_interface/SimpleTransmission</type>
-      <joint name="${prefix}_joint_r2">
-        <hardwareInterface>hardware_interface/PositionJointInterface</hardwareInterface>
-      </joint>
-      <actuator name="${prefix}_motor_r2">
-        <hardwareInterface>hardware_interface/PositionJointInterface</hardwareInterface>
-        <mechanicalReduction>1</mechanicalReduction>
-      </actuator>
-    </transmission>-->
     <!-- Right Link 2 -->
     <link name="${prefix}_link_r2">
@@ -213,14 +193,4 @@
       </plugin>
     </gazebo>
-<!--    <transmission name="${prefix}_transmission_l1">
-      <type>transmission_interface/SimpleTransmission</type>
-      <joint name="${prefix}_joint_l1">
-        <hardwareInterface>hardware_interface/PositionJointInterface</hardwareInterface>
-      </joint>
-      <actuator name="${prefix}_motor_l1">
-        <hardwareInterface>hardware_interface/PositionJointInterface</hardwareInterface>
-        <mechanicalReduction>1</mechanicalReduction>
-      </actuator>
-    </transmission>-->
     <!-- Left Link 1 -->
     <link name="${prefix}_link_l1">
@@ -274,14 +244,4 @@
       </plugin>
     </gazebo>
-<!--    <transmission name="${prefix}_transmission_l2">
-      <type>transmission_interface/SimpleTransmission</type>
-      <joint name="${prefix}_joint_l2">
-        <hardwareInterface>hardware_interface/PositionJointInterface</hardwareInterface>
-      </joint>
-      <actuator name="${prefix}_motor_l2">
-        <hardwareInterface>hardware_interface/PositionJointInterface</hardwareInterface>
-        <mechanicalReduction>1</mechanicalReduction>
-      </actuator>
-    </transmission>-->
     <!-- Left Link 2 -->
     <link name="${prefix}_link_l2">
